File: firmware/eagle/Knightr0's Gambit/Motherboard.sch (EAGLE design)
At the start: 20 parts, among them IC1 7805T, Q1 BUZ10, X1 22-23-2021, X2 22-23-2031, X3 22-23-2031, X4 22-23-2041, X5 22-23-2041, X6 22-23-2041, X7 22-23-2021, X8 22-23-2021

Commit message: update eagle files
Parts:
- added R7, R8: (no value), rcl:R-EU_R0603
- added X10, X9: 22-23-2021, con-molex:22-23-2021
- D1: device adafruit:SCHOTTKY-DIODECB417-15 -> adafruit:SCHOTTKY-DIODEDO41
Connections:
- removed net X_ENDSTOP: BOARD1.D18, R3.1, X7-2.S
- removed net Y_ENDSTOP: BOARD1.D19, R4.1, X8-2.S
- new net X_ENDSTOP_MAX: BOARD1.VP, R7.1, X9-2.S
- new net X_ENDSTOP_MIN: BOARD1.VN, R6.1, X8-2.S
- new net Y_ENDSTOP_MAX: BOARD1.D34, R5.1, X10-2.S
- new net Y_ENDSTOP_MIN: BOARD1.D35, R4.1, X7-2.S
- net +12V: now also R1.2, X2-1.S; no longer R6.2
- net 3.3V: now also X10-1.S, X9-1.S
- net AGND: now also R6.2, R7.2, R8.2; no longer R3.2
- net DRAIN: now also R3.2; no longer R2.2
- net MAGNET: now also R2.1; no longer R1.1
- net N$10: now also R2.2; no longer R1.2
- net N$12: now also R1.1; no longer R6.1, X2-1.S
- net N$9: now also R3.1; no longer R2.1
- net TIMER_BUTTON: now also R8.1; no longer R5.1
Other:
- moved on the sheet: D1, R1, R2, R3, R4, R5, R6, X2-1, X2-2, X2-3, X7-1, X7-2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

Commit message: Updated pcb files
Parts:
- removed U$1, U$2: STEPPER-MOTOR-EASY-DRIVER, Ultrasonic Sensor:STEPPER-MOTOR-EASY-DRIVER
- added C1: 100uF, rcl:CPOL-USB45181A
- added D2, D3: (no value), SparkFun-LED:LED0603
- added R10: 270, rcl:R-EU_R0603
- added R9: 1.2k, rcl:R-EU_R0603
- added S1: (no value), adafruit:EG1218S
- added U1, U2: A4988_STEPPER_MOTOR_DRIVER_CARRIER, A4988_STEPPER_MOTOR_DRIVER_CARRIER:A4988_STEPPER_MOTOR_DRIVER_CARRIER
- added X11: 22-23-2031, con-molex:22-23-2031
- R1: value (none) -> 100
- R2, R4, R5, R6, R7, R8: value (none) -> 1.2k
Connections:
- removed net ENA: BOARD1.D4, U$1.ENA, U$2.ENA
- removed net PFD: U$1.PFD, U$2.PFD
- removed net RST: BOARD1.D2, U$1.RST, U$2.RST
- removed net SLP: BOARD1.D15, U$1.SLP, U$2.SLP
- new net INDICATOR_LED: BOARD1.D21, R10.2
- new net N$13: S1.P, X3-1.S
- new net N$22: U1.2A, X6-3.S
- new net N$23: U1.2B, X6-4.S
- new net X_ENA: BOARD1.D13, U1.!ENABLE
- new net X_MS3: BOARD1.D4, U1.MS3
- new net X_SLP/RST: BOARD1.D12, U1.!RESET, U1.!SLEEP
- new net Y_ENA: BOARD1.D26, U2.!ENABLE
- new net Y_MS3: BOARD1.D19, U2.MS3
- new net Y_SLP/RST: BOARD1.D25, U2.!RESET, U2.!SLEEP
- net +12V: now also C1.+, U1.VMOT, U2.VMOT, X11-3.S; no longer U$1.M+, U$2.M+
- net +5V: now also R9.2, U1.VDD, U2.VDD
- net AGND: now also C1.-, D2.C, D3.C, S1.S, U1.GND, U2.GND, X11-1.S; no longer U$1.GND, U$1.GND.2, U$2.GND, U$2.GND.2, X3-1.S
- net N$1: now also U2.1A, X5-2.S; no longer U$1.A.1, X6-1.S
- net N$2: now also U2.1B, X5-1.S; no longer U$1.A.2, X6-2.S
- net N$3: now also U2.2A, X5-3.S; no longer U$1.B.1, X6-3.S
- net N$4: now also U2.2B, X5-4.S; no longer U$1.B.2, X6-4.S
- net N$5: now also U1.1A, X6-2.S; no longer U$2.A.1, X5-1.S
- net N$6: now also U1.1B, X6-1.S; no longer U$2.A.2, X5-2.S
- net N$7: now also D2.A, R9.1; no longer U$2.B.1, X5-3.S
- net N$8: now also D3.A, R10.1; no longer U$2.B.2, X5-4.S
- net TIMER_BUTTON: now also BOARD1.D22; no longer BOARD1.D21
- net X_DIR: now also U1.DIR; no longer U$1.DIR
- net X_MS1: now also BOARD1.D15, U1.MS1; no longer BOARD1.D13, U$1.MS1
- net X_MS2: now also BOARD1.D2, U1.MS2; no longer BOARD1.D12, U$1.MS2
- net X_STEP: now also U1.STEP; no longer U$1.STER
- net Y_DIR: now also U2.DIR; no longer U$2.DIR
- net Y_MS1: now also BOARD1.D5, U2.MS1; no longer BOARD1.D26, U$2.MS1
- net Y_MS2: now also BOARD1.D18, U2.MS2; no longer BOARD1.D25, U$2.MS2
- net Y_STEP: now also U2.STEP; no longer U$2.STER
Other:
- note added: "Power In"
- note added: "Power Out"
- moved on the sheet: BOARD1, D1, IC1, Q1, R1, R2, R3, R5, R7, X10-1, X10-2, X2-1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
